Commit message: Update yahboom_xgo_rviz.urdf

File: urdf/yahboom_xgo_rviz.urdf (robot description, URDF)
Before this commit: robot xgo, 17 links, 16 joints
Links:
- link base_link: geometry collision mesh filename=package://yahboom_description/meshes/XGO/base_link.STL; visual mesh filename=package://yahboom_description/meshes/XGO/base_link.STL
- link camera_link: geometry collision mesh filename=package://yahboom_description/meshes/XGO/camera_link.STL; visual mesh filename=package://yahboom_description/meshes/XGO/camera_link.STL
- link laser_link: geometry collision mesh filename=package://yahboom_description/meshes/XGO/laser_link.STL; visual mesh filename=package://yahboom_description/meshes/XGO/laser_link.STL
- link lf_hip_link: geometry collision mesh filename=package://yahboom_description/meshes/XGO/lf_hip_link.STL; visual mesh filename=package://yahboom_description/meshes/XGO/lf_hip_link.STL
- link lf_lower_leg_link: geometry collision mesh filename=package://yahboom_description/meshes/XGO/lf_lower_leg_link.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; visual mesh filename=package://yahboom_description/meshes/XGO/lf_lower_leg_link.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
- link lf_upper_leg_link: geometry collision mesh filename=package://yahboom_description/meshes/XGO/lf_upper_leg_link.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; visual mesh filename=package://yahboom_description/meshes/XGO/lf_upper_leg_link.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
- link lh_hip_link: geometry collision mesh filename=package://yahboom_description/meshes/XGO/lh_hip_link.STL; visual mesh filename=package://yahboom_description/meshes/XGO/lh_hip_link.STL
- link lh_lower_leg_link: geometry collision mesh filename=package://yahboom_description/meshes/XGO/lh_lower_leg_link.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; visual mesh filename=package://yahboom_description/meshes/XGO/lh_lower_leg_link.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
- link lh_upper_leg_link: geometry collision mesh filename=package://yahboom_description/meshes/XGO/lh_upper_leg_link.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; visual mesh filename=package://yahboom_description/meshes/XGO/lh_upper_leg_link.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
- link rf_hip_link: geometry collision mesh filename=package://yahboom_description/meshes/XGO/rf_hip_link.STL; visual mesh filename=package://yahboom_description/meshes/XGO/rf_hip_link.STL
- link rf_lower_leg_link: geometry collision mesh filename=package://yahboom_description/meshes/XGO/rf_lower_leg_link.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; visual mesh filename=package://yahboom_description/meshes/XGO/rf_lower_leg_link.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
- link rf_upper_leg_link: geometry collision mesh filename=package://yahboom_description/meshes/XGO/rf_upper_leg_link.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; visual mesh filename=package://yahboom_description/meshes/XGO/rf_upper_leg_link.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
- link rh_hip_link: geometry collision mesh filename=package://yahboom_description/meshes/XGO/rh_hip_link.STL; visual mesh filename=package://yahboom_description/meshes/XGO/rh_hip_link.STL
- link rh_lower_leg_link: geometry collision mesh filename=package://yahboom_description/meshes/XGO/rh_lower_leg_link.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; visual mesh filename=package://yahboom_description/meshes/XGO/rh_lower_leg_link.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
- link rh_upper_leg_link: geometry collision mesh filename=package://yahboom_description/meshes/XGO/rh_upper_leg_link.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; visual mesh filename=package://yahboom_description/meshes/XGO/rh_upper_leg_link.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

Commit message: Update yahboom_xgo_rviz.urdf

File: urdf/yahboom_xgo_rviz.urdf (robot description, URDF)
Before this commit: robot xgo, 17 links, 16 joints
Links:
- removed link imu_link
Joints:
- removed joint imu_Joint
