Commit message: Update yahboom_xgo_rviz.xacro

File: urdf/yahboom_xgo_rviz.xacro (robot description, xacro)
@@ -33,5 +33,5 @@
       <geometry>
         <mesh
-          filename="file:///home/yahboom/cartoros2/src/yahboom_description/meshes/XGO/base_link.STL" />
+          filename="package://yahboom_description/meshes/XGO/base_link.STL" />
       </geometry>
       <material
@@ -47,5 +47,5 @@
       <geometry>
         <mesh
-          filename="file:///home/yahboom/cartoros2/src/yahboom_description/meshes/XGO/base_link.STL" />
+          filename="package://yahboom_description/meshes/XGO/base_link.STL" />
       </geometry>
     </collision>
@@ -73,19 +73,19 @@
       <geometry>
         <mesh
-          filename="file:///home/yahboom/cartoros2/src/yahboom_description/meshes/XGO/lf_hip_link.STL" />
-      </geometry>
-      <material
-        name="">
-        <color
-          rgba="0.898039215686275 0.917647058823529 0.929411764705882 1" />
-      </material>
-    </visual>
-    <collision>
-      <origin
-        xyz="0 0 0"
-        rpy="0 0 0" />
-      <geometry>
-        <mesh
-          filename="file:///home/yahboom/cartoros2/src/yahboom_description/meshes/XGO/lf_hip_link.STL" />
+          filename="package://yahboom_description/meshes/XGO/lf_hip_link.STL" />
+      </geometry>
+      <material
+        name="">
+        <color
+          rgba="0.898039215686275 0.917647058823529 0.929411764705882 1" />
+      </material>
+    </visual>
+    <collision>
+      <origin
+        xyz="0 0 0"
+        rpy="0 0 0" />
+      <geometry>
+        <mesh
+          filename="package://yahboom_description/meshes/XGO/lf_hip_link.STL" />
       </geometry>
     </collision>
@@ -127,19 +127,19 @@
       <geometry>
         <mesh
-          filename="file:///home/yahboom/cartoros2/src/yahboom_description/meshes/XGO/lf_upper_leg_link.STL" />
-      </geometry>
-      <material
-        name="">
-        <color
-          rgba="0.898039215686275 0.917647058823529 0.929411764705882 1" />
-      </material>
-    </visual>
-    <collision>
-      <origin
-        xyz="0 0 0"
-        rpy="0 0 0" />
-      <geometry>
-        <mesh
-          filename="file:///home/yahboom/cartoros2/src/yahboom_description/meshes/XGO/lf_upper_leg_link.STL" />
+          filename="package://yahboom_description/meshes/XGO/lf_upper_leg_link.STL" />
+      </geometry>
+      <material
+        name="">
+        <color
+          rgba="0.898039215686275 0.917647058823529 0.929411764705882 1" />
+      </material>
+    </visual>
+    <collision>
+      <origin
+        xyz="0 0 0"
+        rpy="0 0 0" />
+      <geometry>
+        <mesh
+          filename="package://yahboom_description/meshes/XGO/lf_upper_leg_link.STL" />
       </geometry>
     </collision>
@@ -181,19 +181,19 @@
       <geometry>
         <mesh
-          filename="file:///home/yahboom/cartoros2/src/yahboom_description/meshes/XGO/lf_lower_leg_link.STL" />
-      </geometry>
-      <material
-        name="">
-        <color
-          rgba="0.898039215686275 0.917647058823529 0.929411764705882 1" />
-      </material>
-    </visual>
-    <collision>
-      <origin
-        xyz="0 0 0"
-        rpy="0 0 0" />
-      <geometry>
-        <mesh
-          filename="file:///home/yahboom/cartoros2/src/yahboom_description/meshes/XGO/lf_lower_leg_link.STL" />
+          filename="package://yahboom_description/meshes/XGO/lf_lower_leg_link.STL" />
+      </geometry>
+      <material
+        name="">
+        <color
+          rgba="0.898039215686275 0.917647058823529 0.929411764705882 1" />
+      </material>
+    </visual>
+    <collision>
+      <origin
+        xyz="0 0 0"
+        rpy="0 0 0" />
+      <geometry>
+        <mesh
+          filename="package://yahboom_description/meshes/XGO/lf_lower_leg_link.STL" />
       </geometry>
     </collision>
@@ -235,19 +235,19 @@
       <geometry>
         <mesh
-          filename="file:///home/yahboom/cartoros2/src/yahboom_description/meshes/XGO/rf_hip_link.STL" />
-      </geometry>
-      <material
-        name="">
-        <color
-          rgba="0.898039215686275 0.917647058823529 0.929411764705882 1" />
-      </material>
-    </visual>
-    <collision>
-      <origin
-        xyz="0 0 0"
-        rpy="0 0 0" />
-      <geometry>
-        <mesh
-          filename="file:///home/yahboom/cartoros2/src/yahboom_description/meshes/XGO/rf_hip_link.STL" />
+          filename="package://yahboom_description/meshes/XGO/rf_hip_link.STL" />
+      </geometry>
+      <material
+        name="">
+        <color
+          rgba="0.898039215686275 0.917647058823529 0.929411764705882 1" />
+      </material>
+    </visual>
+    <collision>
+      <origin
+        xyz="0 0 0"
+        rpy="0 0 0" />
+      <geometry>
+        <mesh
+          filename="package://yahboom_description/meshes/XGO/rf_hip_link.STL" />
       </geometry>
     </collision>
@@ -289,19 +289,19 @@
       <geometry>
         <mesh
-          filename="file:///home/yahboom/cartoros2/src/yahboom_description/meshes/XGO/rf_upper_leg_link.STL" />
-      </geometry>
-      <material
-        name="">
-        <color
-          rgba="0.898039215686275 0.917647058823529 0.929411764705882 1" />
-      </material>
-    </visual>
-    <collision>
-      <origin
-        xyz="0 0 0"
-        rpy="0 0 0" />
-      <geometry>
-        <mesh
-          filename="file:///home/yahboom/cartoros2/src/yahboom_description/meshes/XGO/rf_upper_leg_link.STL" />
+          filename="package://yahboom_description/meshes/XGO/rf_upper_leg_link.STL" />
+      </geometry>
+      <material
+        name="">
+        <color
+          rgba="0.898039215686275 0.917647058823529 0.929411764705882 1" />
+      </material>
+    </visual>
+    <collision>
+      <origin
+        xyz="0 0 0"
+        rpy="0 0 0" />
+      <geometry>
+        <mesh
+          filename="package://yahboom_description/meshes/XGO/rf_upper_leg_link.STL" />
       </geometry>
     </collision>
@@ -343,19 +343,19 @@
       <geometry>
         <mesh
-          filename="file:///home/yahboom/cartoros2/src/yahboom_description/meshes/XGO/rf_lower_leg_link.STL" />
-      </geometry>
-      <material
-        name="">
-        <color
-          rgba="0.898039215686275 0.917647058823529 0.929411764705882 1" />
-      </material>
-    </visual>
-    <collision>
-      <origin
-        xyz="0 0 0"
-        rpy="0 0 0" />
-      <geometry>
-        <mesh
-          filename="file:///home/yahboom/cartoros2/src/yahboom_description/meshes/XGO/rf_lower_leg_link.STL" />
+          filename="package://yahboom_description/meshes/XGO/rf_lower_leg_link.STL" />
+      </geometry>
+      <material
+        name="">
+        <color
+          rgba="0.898039215686275 0.917647058823529 0.929411764705882 1" />
+      </material>
+    </visual>
+    <collision>
+      <origin
+        xyz="0 0 0"
+        rpy="0 0 0" />
+      <geometry>
+        <mesh
+          filename="package://yahboom_description/meshes/XGO/rf_lower_leg_link.STL" />
       </geometry>
     </collision>
@@ -397,19 +397,19 @@
       <geometry>
         <mesh
-          filename="file:///home/yahboom/cartoros2/src/yahboom_description/meshes/XGO/lh_hip_link.STL" />
-      </geometry>
-      <material
-        name="">
-        <color
-          rgba="0.898039215686275 0.917647058823529 0.929411764705882 1" />
-      </material>
-    </visual>
-    <collision>
-      <origin
-        xyz="0 0 0"
-        rpy="0 0 0" />
-      <geometry>
-        <mesh
-          filename="file:///home/yahboom/cartoros2/src/yahboom_description/meshes/XGO/lh_hip_link.STL" />
+          filename="package://yahboom_description/meshes/XGO/lh_hip_link.STL" />
+      </geometry>
+      <material
+        name="">
+        <color
+          rgba="0.898039215686275 0.917647058823529 0.929411764705882 1" />
+      </material>
+    </visual>
+    <collision>
+      <origin
+        xyz="0 0 0"
+        rpy="0 0 0" />
+      <geometry>
+        <mesh
+          filename="package://yahboom_description/meshes/XGO/lh_hip_link.STL" />
       </geometry>
     </collision>
@@ -451,19 +451,19 @@
       <geometry>
         <mesh
-          filename="file:///home/yahboom/cartoros2/src/yahboom_description/meshes/XGO/lh_upper_leg_link.STL" />
-      </geometry>
-      <material
-        name="">
-        <color
-          rgba="0.898039215686275 0.917647058823529 0.929411764705882 1" />
-      </material>
-    </visual>
-    <collision>
-      <origin
-        xyz="0 0 0"
-        rpy="0 0 0" />
-      <geometry>
-        <mesh
-          filename="file:///home/yahboom/cartoros2/src/yahboom_description/meshes/XGO/lh_upper_leg_link.STL" />
+          filename="package://yahboom_description/meshes/XGO/lh_upper_leg_link.STL" />
+      </geometry>
+      <material
+        name="">
+        <color
+          rgba="0.898039215686275 0.917647058823529 0.929411764705882 1" />
+      </material>
+    </visual>
+    <collision>
+      <origin
+        xyz="0 0 0"
+        rpy="0 0 0" />
+      <geometry>
+        <mesh
+          filename="package://yahboom_description/meshes/XGO/lh_upper_leg_link.STL" />
       </geometry>
     </collision>
@@ -505,19 +505,19 @@
       <geometry>
         <mesh
-          filename="file:///home/yahboom/cartoros2/src/yahboom_description/meshes/XGO/lh_lower_leg_link.STL" />
-      </geometry>
-      <material
-        name="">
-        <color
-          rgba="0.898039215686275 0.917647058823529 0.929411764705882 1" />
-      </material>
-    </visual>
-    <collision>
-      <origin
-        xyz="0 0 0"
-        rpy="0 0 0" />
-      <geometry>
-        <mesh
-          filename="file:///home/yahboom/cartoros2/src/yahboom_description/meshes/XGO/lh_lower_leg_link.STL" />
+          filename="package://yahboom_description/meshes/XGO/lh_lower_leg_link.STL" />
+      </geometry>
+      <material
+        name="">
+        <color
+          rgba="0.898039215686275 0.917647058823529 0.929411764705882 1" />
+      </material>
+    </visual>
+    <collision>
+      <origin
+        xyz="0 0 0"
+        rpy="0 0 0" />
+      <geometry>
+        <mesh
+          filename="package://yahboom_description/meshes/XGO/lh_lower_leg_link.STL" />
       </geometry>
     </collision>
@@ -559,19 +559,19 @@
       <geometry>
         <mesh
-          filename="file:///home/yahboom/cartoros2/src/yahboom_description/meshes/XGO/rh_hip_link.STL" />
-      </geometry>
-      <material
-        name="">
-        <color
-          rgba="0.898039215686275 0.917647058823529 0.929411764705882 1" />
-      </material>
-    </visual>
-    <collision>
-      <origin
-        xyz="0 0 0"
-        rpy="0 0 0" />
-      <geometry>
-        <mesh
-          filename="file:///home/yahboom/cartoros2/src/yahboom_description/meshes/XGO/rh_hip_link.STL" />
+          filename="package://yahboom_description/meshes/XGO/rh_hip_link.STL" />
+      </geometry>
+      <material
+        name="">
+        <color
+          rgba="0.898039215686275 0.917647058823529 0.929411764705882 1" />
+      </material>
+    </visual>
+    <collision>
+      <origin
+        xyz="0 0 0"
+        rpy="0 0 0" />
+      <geometry>
+        <mesh
+          filename="package://yahboom_description/meshes/XGO/rh_hip_link.STL" />
       </geometry>
     </collision>
@@ -613,19 +613,19 @@
       <geometry>
         <mesh
-          filename="file:///home/yahboom/cartoros2/src/yahboom_description/meshes/XGO/rh_upper_leg_link.STL" />
-      </geometry>
-      <material
-        name="">
-        <color
-          rgba="0.898039215686275 0.917647058823529 0.929411764705882 1" />
-      </material>
-    </visual>
-    <collision>
-      <origin
-        xyz="0 0 0"
-        rpy="0 0 0" />
-      <geometry>
-        <mesh
-          filename="file:///home/yahboom/cartoros2/src/yahboom_description/meshes/XGO/rh_upper_leg_link.STL" />
+          filename="package://yahboom_description/meshes/XGO/rh_upper_leg_link.STL" />
+      </geometry>
+      <material
+        name="">
+        <color
+          rgba="0.898039215686275 0.917647058823529 0.929411764705882 1" />
+      </material>
+    </visual>
+    <collision>
+      <origin
+        xyz="0 0 0"
+        rpy="0 0 0" />
+      <geometry>
+        <mesh
+          filename="package://yahboom_description/meshes/XGO/rh_upper_leg_link.STL" />
       </geometry>
     </collision>
@@ -667,19 +667,19 @@
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